File: hardware/motherboard_clean.brd (EAGLE design)
At the start: 118.1 x 76.2 mm, 55 parts

Commit message: Added hardware
Parts:
- removed E$38, E$39, E$9: (no value), 40xx:DIL08
- removed E$40, E$56: (no value), con-molex:22-23-2031
- removed E$41: (no value), relay:351
- removed E$42, E$48: (no value), 74xx-eu:DIL08
- removed E$43, E$49: (no value), diode:D-7.5
- removed E$44, E$45, E$46, E$47, E$50, E$52, E$54, E$55: (no value), BeagleBone_Black_Wireless:0207/7
- removed E$51: (no value), jumper:JP1
- E$10: device relay:351 -> BeagleBone_Black_Wireless:0207/10
- moved E$10 115.2 mm to (168.9, 73.7)
- moved E$27 75.0 mm to (6.73, 53.1)
- moved E$28 75.0 mm to (-3.81, 57.1)
- moved E$30 75.0 mm to (10.2, 62.2)
- moved E$35 75.0 mm to (-8.89, 57.1)
- moved E$36 75.0 mm to (-12.1, 64.1)
- moved E$25 75.0 mm to (2.54, 61.0)
- moved E$26 75.0 mm to (1.40, 51.8)
- moved E$29 75.0 mm to (-5.08, 50.8)
- moved E$31 75.0 mm to (3.81, 67.3)
- moved E$32 75.0 mm to (-5.97, 68.6)
- moved E$33 75.0 mm to (-1.27, 69.8)
- moved E$34 75.0 mm to (-6.35, 59.7)
- moved E$14 4.58 mm to (50.8, 26.7)
- moved E$6 4.02 mm to (85.1, 48.3)
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Connections:
- removed net +3V: E$13.3, E$15.+, E$37.+, E$5.9
- removed net +5V: E$11.5, E$12.C, E$14.+, E$48.8, E$5.8, E$51.1, E$52.2, E$55.2, E$6.1
- removed net +5V_JMP: E$1.11, E$1.32, E$3.1, E$40.2, E$51.2
- removed net GND: E$1.12, E$1.31, E$10.16, E$11.1, E$11.3, E$11.7, E$13.2, E$14.-, E$16.3, E$17.1, E$18.11, E$2.1, E$2.19, E$21.2, E$22.1, E$3.2, E$37.-, E$4.2, E$40.3, E$48.5, E$5.10, E$56.1, E$7.1, E$7.11, E$7.4, E$7.6, E$7.9, E$8.-
- removed net S$32: E$41.1
- removed net S$46: E$46.2
- removed net S$47: E$41.S2, E$42.2, E$43.C
- removed net S$49: E$48.3, E$49.A, E$50.1
- removed net S$50: E$42.3, E$43.A, E$44.1
- removed net S$52: E$10.S1, E$48.2, E$49.C
- removed net S$53: E$1.22, E$54.2
- removed net S$55: E$1.30, E$2.11
- removed net S$60: E$41.P1
- removed net S$61: E$41.P2
- removed net S$63: E$12.A, E$15.-, E$16.2
- new net S$16: E$1.31, E$4.2
- new net S$21: E$2.18
- new net S$23: E$2.16
- new net S$24: E$2.15
- new net S$25: E$2.14
- new net S$3: E$2.4
- new net S$31: E$1.11, E$1.32, E$3.1
- new net S$33: E$1.40
- new net S$71: E$13.3, E$15.+, E$37.+
- new net S$72: E$1.9
- new net S$86: E$17.1, E$18.11
- new net S$88: E$19.+
- net S$1: now also E$2.2; no longer E$20.-, E$7.10
- net S$10: no longer E$2.3
- net S$11: no longer E$2.4
- net S$12: no longer E$2.5
- net S$13: no longer E$2.6
- net S$14: no longer E$2.7
- net S$19: no longer E$2.14
- net S$2: now also E$2.3; no longer E$38.1, E$38.8, E$39.1, E$39.2, E$39.8, E$9.8
- net S$22: now also E$2.17; no longer E$38.5, E$39.5, E$9.5
- net S$26: no longer E$2.15
- net S$27: no longer E$2.16
- net S$28: no longer E$2.17
- net S$29: no longer E$2.18
- net S$30: now also E$1.1; no longer E$1.10, E$40.1
- net S$34: now also E$1.12, E$3.2; no longer E$41.16
- net S$35: now also E$1.39; no longer E$41.O2, E$45.2
- net S$4: now also E$2.5; no longer E$39.6
- net S$43: now also E$5.8, E$6.1; no longer E$1.21, E$48.6, E$55.1
- net S$44: now also E$2.11; no longer E$42.8, E$45.1, E$47.1
- net S$45: now also E$1.30; no longer E$41.O1, E$46.1
- net S$5: now also E$2.6; no longer E$38.6
- net S$56: now also E$1.27; no longer E$10.S2, E$50.2
- net S$57: now also E$1.28; no longer E$41.S1, E$44.2
- net S$59: now also E$1.29; no longer E$10.O2, E$54.1
- net S$6: now also E$2.7; no longer E$9.6
- net S$64: now also E$1.8; no longer E$42.6, E$47.2
- net S$65: now also E$11.5, E$12.C; no longer E$1.23, E$10.1
- net S$66: now also E$12.A, E$15.-, E$16.2; no longer E$10.P1, E$56.3
- net S$67: now also E$11.3, E$14.-; no longer E$10.P2, E$56.2
- net S$68: now also E$11.1, E$11.7; no longer E$38.2, E$38.3, E$38.4, E$38.7, E$39.3, E$39.4, E$39.7, E$9.1, E$9.2, E$9.3, E$9.4, E$9.7
- net S$69: now also E$5.9; no longer E$10.O1, E$52.1
- net S$7: no longer E$1.39
- net S$77: no longer E$1.8
- net S$78: no longer E$1.9
- net S$8: no longer E$1.40
- net S$80: now also E$1.10; no longer E$1.1, E$7.3
- net S$84: no longer E$2.21
- net S$85: no longer E$2.20
- net S$89: no longer E$19.+
- net S$9: no longer E$2.2
Routing:
- net +5V: track 103.2 -> 0.00 mm, vias 4 -> 0
- net S$55: track 96.5 -> 5.08 mm, vias 4 -> 2
- net S$68: track 77.8 -> 10.2 mm, vias 1 -> 0
- net +5V_JMP: track 59.3 -> 0.00 mm, vias 1 -> 0
- net S$22: track 63.5 -> 5.08 mm, vias 7 -> 1
- net S$2: track 58.4 -> 5.24 mm
- net S$7: track 62.1 -> 11.5 mm, vias 5 -> 1
- net S$19: track 58.4 -> 8.89 mm, vias 2 -> 1
- net S$31: track 0.00 -> 49.3 mm, vias 0 -> 1
- net S$8: track 61.0 -> 12.8 mm, vias 3 -> 1
- net S$26: track 55.9 -> 7.62 mm, vias 2 -> 1
- net S$27: track 53.3 -> 6.35 mm, vias 2 -> 1
- net S$28: track 50.8 -> 5.08 mm, vias 2 -> 1
- net S$4: track 53.3 -> 7.73 mm
- net S$29: track 48.3 -> 3.81 mm, vias 2 -> 1
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Other:
- board size 118.1 x 76.2 mm -> 116.8 x 76.2 mm
- board text removed: "+3V"
- board text removed: "SCL"
- board text removed: "SDA"
